Commit message: temp

File: urdf/model.urdf (robot description, URDF)
Before this commit: robot hex_robot, 8 links, 7 joints
Links:
- removed link link_4
- removed link link_5
- removed link link_6
- removed link link_7
- added link link_1_caster_0, mass 0.0059; collision sphere radius=0.025; visual sphere radius=0.025
- added link link_1_caster_1, mass 0.0059; collision sphere radius=0.025; visual sphere radius=0.025
- added link link_1_caster_2, mass 0.0059; collision sphere radius=0.025; visual sphere radius=0.025
- added link link_1_caster_3, mass 0.0059; collision sphere radius=0.025; visual sphere radius=0.025
- added link link_1_caster_4, mass 0.0059; collision sphere radius=0.025; visual sphere radius=0.025
- added link link_1_caster_5, mass 0.0059; collision sphere radius=0.025; visual sphere radius=0.025
- added link link_1_caster_6, mass 0.0059; collision sphere radius=0.025; visual sphere radius=0.025
- added link link_1_caster_7, mass 0.0059; collision sphere radius=0.025; visual sphere radius=0.025
- added link link_2_caster_0, mass 0.0059; collision sphere radius=0.025; visual sphere radius=0.025
- added link link_2_caster_1, mass 0.0059; collision sphere radius=0.025; visual sphere radius=0.025
- added link link_2_caster_2, mass 0.0059; collision sphere radius=0.025; visual sphere radius=0.025
- added link link_2_caster_3, mass 0.0059; collision sphere radius=0.025; visual sphere radius=0.025
- added link link_2_caster_4, mass 0.0059; collision sphere radius=0.025; visual sphere radius=0.025
- added link link_2_caster_5, mass 0.0059; collision sphere radius=0.025; visual sphere radius=0.025
- added link link_2_caster_6, mass 0.0059; collision sphere radius=0.025; visual sphere radius=0.025
- added link link_2_caster_7, mass 0.0059; collision sphere radius=0.025; visual sphere radius=0.025
- added link link_3_caster_0, mass 0.0059; collision sphere radius=0.025; visual sphere radius=0.025
- added link link_3_caster_1, mass 0.0059; collision sphere radius=0.025; visual sphere radius=0.025
- added link link_3_caster_2, mass 0.0059; collision sphere radius=0.025; visual sphere radius=0.025
- added link link_3_caster_3, mass 0.0059; collision sphere radius=0.025; visual sphere radius=0.025
- added link link_3_caster_4, mass 0.0059; collision sphere radius=0.025; visual sphere radius=0.025
- added link link_3_caster_5, mass 0.0059; collision sphere radius=0.025; visual sphere radius=0.025
- added link link_3_caster_6, mass 0.0059; collision sphere radius=0.025; visual sphere radius=0.025
- added link link_3_caster_7, mass 0.0059; collision sphere radius=0.025; visual sphere radius=0.025
- link base_link: mass 5.0 -> 17.7649882169949; geometry collision mesh filename=package://hex_ros_urdf_trigger_a/meshes/base_link.dae; visual mesh filename=package://hex_ros_urdf_trigger_a/meshes/base_link.dae
- link link_1: mass 2.0 -> 1.62479279397676; geometry visual mesh filename=package://hex_ros_urdf_trigger_a/meshes/link_1.dae
- link link_2: mass 3.0 -> 1.62479279397676; geometry visual mesh filename=package://hex_ros_urdf_trigger_a/meshes/link_2.dae
- link link_3: mass 1.5 -> 1.62479279397676; geometry visual mesh filename=package://hex_ros_urdf_trigger_a/meshes/link_3.dae
Joints:
- removed joint joint_4
- removed joint joint_5
- removed joint joint_6
- removed joint joint_7
- added joint joint_1_caster_0: type continuous, parent link_1, child link_1_caster_0, origin xyz=-0.04 0.075 0.0 rpy=0 0 0, axis 0 0 1
- added joint joint_1_caster_1: type continuous, parent link_1, child link_1_caster_1, origin xyz=-0.04 0.053 0.053 rpy=0 0 0, axis 0 -0.707107 0.707107
- added joint joint_1_caster_2: type continuous, parent link_1, child link_1_caster_2, origin xyz=-0.04 0.0 0.075 rpy=0 0 0, axis 0 -1 0
- added joint joint_1_caster_3: type continuous, parent link_1, child link_1_caster_3, origin xyz=-0.04 -0.053 0.053 rpy=0 0 0, axis 0 -0.707107 -0.707107
- added joint joint_1_caster_4: type continuous, parent link_1, child link_1_caster_4, origin xyz=-0.04 -0.075 0.0 rpy=0 0 0, axis 0 0 -1
- added joint joint_1_caster_5: type continuous, parent link_1, child link_1_caster_5, origin xyz=-0.04 -0.053 -0.053 rpy=0 0 0, axis 0 0.707107 -0.707107
- added joint joint_1_caster_6: type continuous, parent link_1, child link_1_caster_6, origin xyz=-0.04 0.0 -0.075 rpy=0 0 0, axis 0 1 0
- added joint joint_1_caster_7: type continuous, parent link_1, child link_1_caster_7, origin xyz=-0.04 0.053 -0.053 rpy=0 0 0, axis 0 0.707107 0.707107
- added joint joint_2_caster_0: type continuous, parent link_2, child link_2_caster_0, origin xyz=0.04 0.075 0.0 rpy=0 0 0, axis 0 0 1
- added joint joint_2_caster_1: type continuous, parent link_2, child link_2_caster_1, origin xyz=0.04 0.053 0.053 rpy=0 0 0, axis 0 -0.707107 0.707107
- added joint joint_2_caster_2: type continuous, parent link_2, child link_2_caster_2, origin xyz=0.04 0.0 0.075 rpy=0 0 0, axis 0 -1 0
- added joint joint_2_caster_3: type continuous, parent link_2, child link_2_caster_3, origin xyz=0.04 -0.053 0.053 rpy=0 0 0, axis 0 -0.707107 -0.707107
- added joint joint_2_caster_4: type continuous, parent link_2, child link_2_caster_4, origin xyz=0.04 -0.075 0.0 rpy=0 0 0, axis 0 0 -1
- added joint joint_2_caster_5: type continuous, parent link_2, child link_2_caster_5, origin xyz=0.04 -0.053 -0.053 rpy=0 0 0, axis 0 0.707107 -0.707107
- added joint joint_2_caster_6: type continuous, parent link_2, child link_2_caster_6, origin xyz=0.04 0.0 -0.075 rpy=0 0 0, axis 0 1 0
- added joint joint_2_caster_7: type continuous, parent link_2, child link_2_caster_7, origin xyz=0.04 0.053 -0.053 rpy=0 0 0, axis 0 0.707107 0.707107
- added joint joint_3_caster_0: type continuous, parent link_3, child link_3_caster_0, origin xyz=-0.04 0.075 0.0 rpy=0 0 0, axis 0 0 1
- added joint joint_3_caster_1: type continuous, parent link_3, child link_3_caster_1, origin xyz=-0.04 0.053 0.053 rpy=0 0 0, axis 0 -0.707107 0.707107
- added joint joint_3_caster_2: type continuous, parent link_3, child link_3_caster_2, origin xyz=-0.04 0.0 0.075 rpy=0 0 0, axis 0 -1 0
- added joint joint_3_caster_3: type continuous, parent link_3, child link_3_caster_3, origin xyz=-0.04 -0.053 0.053 rpy=0 0 0, axis 0 -0.707107 -0.707107
- added joint joint_3_caster_4: type continuous, parent link_3, child link_3_caster_4, origin xyz=-0.04 -0.075 0.0 rpy=0 0 0, axis 0 0 -1
- added joint joint_3_caster_5: type continuous, parent link_3, child link_3_caster_5, origin xyz=-0.04 -0.053 -0.053 rpy=0 0 0, axis 0 0.707107 -0.707107
- added joint joint_3_caster_6: type continuous, parent link_3, child link_3_caster_6, origin xyz=-0.04 0.0 -0.075 rpy=0 0 0, axis 0 1 0
- added joint joint_3_caster_7: type continuous, parent link_3, child link_3_caster_7, origin xyz=-0.04 0.053 -0.053 rpy=0 0 0, axis 0 0.707107 0.707107
- joint joint_1: axis 0 0 1 -> -1 0 0; limit lower=-2.967 upper=2.967 effort=100 velocity=1.0 -> lower=0 upper=3 effort=2 velocity=2; origin xyz=0 0 0.05 rpy=0 0 0 -> xyz=0.14475 0.25071 0.103 rpy=0 0 -2.0944; type revolute -> continuous
- joint joint_2: axis 0 1 0 -> 1 0 0; limit lower=-2.094 upper=2.094 effort=100 velocity=1.0 -> lower=0 upper=3 effort=2 velocity=2; origin xyz=0 0 0.2 rpy=0 0 0 -> xyz=0.14475 -0.25071 0.103 rpy=0 0 -1.0472; parent link_1 -> base_link; type revolute -> continuous
- joint joint_3: axis 0 0 1 -> -1 0 0; limit lower=-2.967 upper=2.967 effort=50 velocity=1.0 -> lower=0 upper=3 effort=2 velocity=2; origin xyz=0 0 0.3 rpy=0 0 0 -> xyz=-0.2895 0 0.103 rpy=0 0 0; parent link_2 -> base_link; type revolute -> continuous

Commit message: temp

File: urdf/model.urdf (robot description, URDF)
Before this commit: robot trigger_a, 28 links, 27 joints
Links:
- added link link_1_caster_10, mass 0.0059; collision sphere radius=0.015
- added link link_1_caster_11, mass 0.0059; collision sphere radius=0.015
- added link link_1_caster_12, mass 0.0059; collision sphere radius=0.015
- added link link_1_caster_13, mass 0.0059; collision sphere radius=0.015
- added link link_1_caster_14, mass 0.0059; collision sphere radius=0.015
- added link link_1_caster_15, mass 0.0059; collision sphere radius=0.015
- added link link_1_caster_8, mass 0.0059; collision sphere radius=0.015
- added link link_1_caster_9, mass 0.0059; collision sphere radius=0.015
- added link link_2_caster_10, mass 0.0059; collision sphere radius=0.015
- added link link_2_caster_11, mass 0.0059; collision sphere radius=0.015
- added link link_2_caster_12, mass 0.0059; collision sphere radius=0.015
- added link link_2_caster_13, mass 0.0059; collision sphere radius=0.015
- added link link_2_caster_14, mass 0.0059; collision sphere radius=0.015
- added link link_2_caster_15, mass 0.0059; collision sphere radius=0.015
- added link link_2_caster_8, mass 0.0059; collision sphere radius=0.015
- added link link_2_caster_9, mass 0.0059; collision sphere radius=0.015
- added link link_3_caster_10, mass 0.0059; collision sphere radius=0.015
- added link link_3_caster_11, mass 0.0059; collision sphere radius=0.015
- added link link_3_caster_12, mass 0.0059; collision sphere radius=0.015
- added link link_3_caster_13, mass 0.0059; collision sphere radius=0.015
- added link link_3_caster_14, mass 0.0059; collision sphere radius=0.015
- added link link_3_caster_15, mass 0.0059; collision sphere radius=0.015
- added link link_3_caster_8, mass 0.0059; collision sphere radius=0.015
- added link link_3_caster_9, mass 0.0059; collision sphere radius=0.015
- link link_1_caster_0: geometry collision sphere radius=0.015
- link link_1_caster_1: geometry collision sphere radius=0.015
- link link_1_caster_2: geometry collision sphere radius=0.015
- link link_1_caster_3: geometry collision sphere radius=0.015
- link link_1_caster_4: geometry collision sphere radius=0.015
- link link_1_caster_5: geometry collision sphere radius=0.015
- link link_1_caster_6: geometry collision sphere radius=0.015
- link link_1_caster_7: geometry collision sphere radius=0.015
- link link_2_caster_0: geometry collision sphere radius=0.015
- link link_2_caster_1: geometry collision sphere radius=0.015
- link link_2_caster_2: geometry collision sphere radius=0.015
- link link_2_caster_3: geometry collision sphere radius=0.015
- link link_2_caster_4: geometry collision sphere radius=0.015
- link link_2_caster_5: geometry collision sphere radius=0.015
- link link_2_caster_6: geometry collision sphere radius=0.015
- link link_2_caster_7: geometry collision sphere radius=0.015
- link link_3_caster_0: geometry collision sphere radius=0.015
- link link_3_caster_1: geometry collision sphere radius=0.015
- link link_3_caster_2: geometry collision sphere radius=0.015
- link link_3_caster_3: geometry collision sphere radius=0.015
- link link_3_caster_4: geometry collision sphere radius=0.015
- link link_3_caster_5: geometry collision sphere radius=0.015
- link link_3_caster_6: geometry collision sphere radius=0.015
- link link_3_caster_7: geometry collision sphere radius=0.015
Joints:
- added joint joint_1_caster_10: type continuous, parent link_1, child link_1_caster_10, origin xyz=-0.038 -0.033293458 0.080377519 rpy=0 0 0, axis 0 -0.923880 -0.382683
- added joint joint_1_caster_11: type continuous, parent link_1, child link_1_caster_11, origin xyz=-0.038 -0.080377519 0.033293458 rpy=0 0 0, axis 0 -0.382683 -0.923880
- added joint joint_1_caster_12: type continuous, parent link_1, child link_1_caster_12, origin xyz=-0.038 -0.080377519 -0.033293458 rpy=0 0 0, axis 0 0.382683 -0.923880
- added joint joint_1_caster_13: type continuous, parent link_1, child link_1_caster_13, origin xyz=-0.038 -0.033293458 -0.080377519 rpy=0 0 0, axis 0 0.923880 -0.382683
- added joint joint_1_caster_14: type continuous, parent link_1, child link_1_caster_14, origin xyz=-0.038 0.033293458 -0.080377519 rpy=0 0 0, axis 0 0.923880 0.382683
- added joint joint_1_caster_15: type continuous, parent link_1, child link_1_caster_15, origin xyz=-0.038 0.080377519 -0.033293458 rpy=0 0 0, axis 0 0.382683 0.923880
- added joint joint_1_caster_8: type continuous, parent link_1, child link_1_caster_8, origin xyz=-0.038 0.080377519 0.033293458 rpy=0 0 0, axis 0 -0.382683 0.923880
- added joint joint_1_caster_9: type continuous, parent link_1, child link_1_caster_9, origin xyz=-0.038 0.033293458 0.080377519 rpy=0 0 0, axis 0 -0.923880 0.382683
- added joint joint_2_caster_10: type continuous, parent link_2, child link_2_caster_10, origin xyz=0.038 -0.033293458 0.080377519 rpy=0 0 0, axis 0 -0.923880 -0.382683
- added joint joint_2_caster_11: type continuous, parent link_2, child link_2_caster_11, origin xyz=0.038 -0.080377519 0.033293458 rpy=0 0 0, axis 0 -0.382683 -0.923880
- added joint joint_2_caster_12: type continuous, parent link_2, child link_2_caster_12, origin xyz=0.038 -0.080377519 -0.033293458 rpy=0 0 0, axis 0 0.382683 -0.923880
- added joint joint_2_caster_13: type continuous, parent link_2, child link_2_caster_13, origin xyz=0.038 -0.033293458 -0.080377519 rpy=0 0 0, axis 0 0.923880 -0.382683
- added joint joint_2_caster_14: type continuous, parent link_2, child link_2_caster_14, origin xyz=0.038 0.033293458 -0.080377519 rpy=0 0 0, axis 0 0.923880 0.382683
- added joint joint_2_caster_15: type continuous, parent link_2, child link_2_caster_15, origin xyz=0.038 0.080377519 -0.033293458 rpy=0 0 0, axis 0 0.382683 0.923880
- added joint joint_2_caster_8: type continuous, parent link_2, child link_2_caster_8, origin xyz=0.038 0.080377519 0.033293458 rpy=0 0 0, axis 0 -0.382683 0.923880
- added joint joint_2_caster_9: type continuous, parent link_2, child link_2_caster_9, origin xyz=0.038 0.033293458 0.080377519 rpy=0 0 0, axis 0 -0.923880 0.382683
- added joint joint_3_caster_10: type continuous, parent link_3, child link_3_caster_10, origin xyz=-0.038 -0.033293458 0.080377519 rpy=0 0 0, axis 0 -0.923880 -0.382683
- added joint joint_3_caster_11: type continuous, parent link_3, child link_3_caster_11, origin xyz=-0.038 -0.080377519 0.033293458 rpy=0 0 0, axis 0 -0.382683 -0.923880
- added joint joint_3_caster_12: type continuous, parent link_3, child link_3_caster_12, origin xyz=-0.038 -0.080377519 -0.033293458 rpy=0 0 0, axis 0 0.382683 -0.923880
- added joint joint_3_caster_13: type continuous, parent link_3, child link_3_caster_13, origin xyz=-0.038 -0.033293458 -0.080377519 rpy=0 0 0, axis 0 0.923880 -0.382683
- added joint joint_3_caster_14: type continuous, parent link_3, child link_3_caster_14, origin xyz=-0.038 0.033293458 -0.080377519 rpy=0 0 0, axis 0 0.923880 0.382683
- added joint joint_3_caster_15: type continuous, parent link_3, child link_3_caster_15, origin xyz=-0.038 0.080377519 -0.033293458 rpy=0 0 0, axis 0 0.382683 0.923880
- added joint joint_3_caster_8: type continuous, parent link_3, child link_3_caster_8, origin xyz=-0.038 0.080377519 0.033293458 rpy=0 0 0, axis 0 -0.382683 0.923880
- added joint joint_3_caster_9: type continuous, parent link_3, child link_3_caster_9, origin xyz=-0.038 0.033293458 0.080377519 rpy=0 0 0, axis 0 -0.923880 0.382683
- joint joint_1_caster_0: origin xyz=-0.04 0.075 0.0 rpy=0 0 0 -> xyz=-0.038 0.087 0.0 rpy=0 0 0
- joint joint_1_caster_1: origin xyz=-0.04 0.053 0.053 rpy=0 0 0 -> xyz=-0.038 0.061518290 0.061518290 rpy=0 0 0
- joint joint_1_caster_2: origin xyz=-0.04 0.0 0.075 rpy=0 0 0 -> xyz=-0.038 0.0 0.087 rpy=0 0 0
- joint joint_1_caster_3: origin xyz=-0.04 -0.053 0.053 rpy=0 0 0 -> xyz=-0.038 -0.061518290 0.061518290 rpy=0 0 0
- joint joint_1_caster_4: origin xyz=-0.04 -0.075 0.0 rpy=0 0 0 -> xyz=-0.038 -0.087 0.0 rpy=0 0 0
- joint joint_1_caster_5: origin xyz=-0.04 -0.053 -0.053 rpy=0 0 0 -> xyz=-0.038 -0.061518290 -0.061518290 rpy=0 0 0
- joint joint_1_caster_6: origin xyz=-0.04 0.0 -0.075 rpy=0 0 0 -> xyz=-0.038 0.0 -0.087 rpy=0 0 0
- joint joint_1_caster_7: origin xyz=-0.04 0.053 -0.053 rpy=0 0 0 -> xyz=-0.038 0.061518290 -0.061518290 rpy=0 0 0
- joint joint_2_caster_0: origin xyz=0.04 0.075 0.0 rpy=0 0 0 -> xyz=0.038 0.087 0.0 rpy=0 0 0
- joint joint_2_caster_1: origin xyz=0.04 0.053 0.053 rpy=0 0 0 -> xyz=0.038 0.061518290 0.061518290 rpy=0 0 0
- joint joint_2_caster_2: origin xyz=0.04 0.0 0.075 rpy=0 0 0 -> xyz=0.038 0.0 0.087 rpy=0 0 0
- joint joint_2_caster_3: origin xyz=0.04 -0.053 0.053 rpy=0 0 0 -> xyz=0.038 -0.061518290 0.061518290 rpy=0 0 0
- joint joint_2_caster_4: origin xyz=0.04 -0.075 0.0 rpy=0 0 0 -> xyz=0.038 -0.087 0.0 rpy=0 0 0
- joint joint_2_caster_5: origin xyz=0.04 -0.053 -0.053 rpy=0 0 0 -> xyz=0.038 -0.061518290 -0.061518290 rpy=0 0 0
- joint joint_2_caster_6: origin xyz=0.04 0.0 -0.075 rpy=0 0 0 -> xyz=0.038 0.0 -0.087 rpy=0 0 0
- joint joint_2_caster_7: origin xyz=0.04 0.053 -0.053 rpy=0 0 0 -> xyz=0.038 0.061518290 -0.061518290 rpy=0 0 0
- joint joint_3_caster_0: origin xyz=-0.04 0.075 0.0 rpy=0 0 0 -> xyz=-0.038 0.087 0.0 rpy=0 0 0
- joint joint_3_caster_1: origin xyz=-0.04 0.053 0.053 rpy=0 0 0 -> xyz=-0.038 0.061518290 0.061518290 rpy=0 0 0
- joint joint_3_caster_2: origin xyz=-0.04 0.0 0.075 rpy=0 0 0 -> xyz=-0.038 0.0 0.087 rpy=0 0 0
- joint joint_3_caster_3: origin xyz=-0.04 -0.053 0.053 rpy=0 0 0 -> xyz=-0.038 -0.061518290 0.061518290 rpy=0 0 0
- joint joint_3_caster_4: origin xyz=-0.04 -0.075 0.0 rpy=0 0 0 -> xyz=-0.038 -0.087 0.0 rpy=0 0 0
- joint joint_3_caster_5: origin xyz=-0.04 -0.053 -0.053 rpy=0 0 0 -> xyz=-0.038 -0.061518290 -0.061518290 rpy=0 0 0
- joint joint_3_caster_6: origin xyz=-0.04 0.0 -0.075 rpy=0 0 0 -> xyz=-0.038 0.0 -0.087 rpy=0 0 0
- joint joint_3_caster_7: origin xyz=-0.04 0.053 -0.053 rpy=0 0 0 -> xyz=-0.038 0.061518290 -0.061518290 rpy=0 0 0
