Commit message: temp

File: urdf/model.urdf (robot description, URDF)
Before this commit: robot trigger_a, 52 links, 51 joints
Joints:
- joint joint_1_caster_0: origin xyz=-0.038 0.087 0.0 rpy=0 0 0 -> xyz=-0.0357 0.087 0.0 rpy=0 0 0
- joint joint_1_caster_1: origin xyz=-0.038 0.061518290 0.061518290 rpy=0 0 0 -> xyz=-0.0357 0.061518290 0.061518290 rpy=0 0 0
- joint joint_1_caster_10: origin xyz=-0.038 -0.033293458 0.080377519 rpy=0 0 0 -> xyz=-0.0357 -0.033293458 0.080377519 rpy=0 0 0
- joint joint_1_caster_11: origin xyz=-0.038 -0.080377519 0.033293458 rpy=0 0 0 -> xyz=-0.0357 -0.080377519 0.033293458 rpy=0 0 0
- joint joint_1_caster_12: origin xyz=-0.038 -0.080377519 -0.033293458 rpy=0 0 0 -> xyz=-0.0357 -0.080377519 -0.033293458 rpy=0 0 0
- joint joint_1_caster_13: origin xyz=-0.038 -0.033293458 -0.080377519 rpy=0 0 0 -> xyz=-0.0357 -0.033293458 -0.080377519 rpy=0 0 0
- joint joint_1_caster_14: origin xyz=-0.038 0.033293458 -0.080377519 rpy=0 0 0 -> xyz=-0.0357 0.033293458 -0.080377519 rpy=0 0 0
- joint joint_1_caster_15: origin xyz=-0.038 0.080377519 -0.033293458 rpy=0 0 0 -> xyz=-0.0357 0.080377519 -0.033293458 rpy=0 0 0
- joint joint_1_caster_2: origin xyz=-0.038 0.0 0.087 rpy=0 0 0 -> xyz=-0.0357 0.0 0.087 rpy=0 0 0
- joint joint_1_caster_3: origin xyz=-0.038 -0.061518290 0.061518290 rpy=0 0 0 -> xyz=-0.0357 -0.061518290 0.061518290 rpy=0 0 0
- joint joint_1_caster_4: origin xyz=-0.038 -0.087 0.0 rpy=0 0 0 -> xyz=-0.0357 -0.087 0.0 rpy=0 0 0
- joint joint_1_caster_5: origin xyz=-0.038 -0.061518290 -0.061518290 rpy=0 0 0 -> xyz=-0.0357 -0.061518290 -0.061518290 rpy=0 0 0
- joint joint_1_caster_6: origin xyz=-0.038 0.0 -0.087 rpy=0 0 0 -> xyz=-0.0357 0.0 -0.087 rpy=0 0 0
- joint joint_1_caster_7: origin xyz=-0.038 0.061518290 -0.061518290 rpy=0 0 0 -> xyz=-0.0357 0.061518290 -0.061518290 rpy=0 0 0
- joint joint_1_caster_8: origin xyz=-0.038 0.080377519 0.033293458 rpy=0 0 0 -> xyz=-0.0357 0.080377519 0.033293458 rpy=0 0 0
- joint joint_1_caster_9: origin xyz=-0.038 0.033293458 0.080377519 rpy=0 0 0 -> xyz=-0.0357 0.033293458 0.080377519 rpy=0 0 0
- joint joint_2_caster_0: origin xyz=0.038 0.087 0.0 rpy=0 0 0 -> xyz=0.0357 0.087 0.0 rpy=0 0 0
- joint joint_2_caster_1: origin xyz=0.038 0.061518290 0.061518290 rpy=0 0 0 -> xyz=0.0357 0.061518290 0.061518290 rpy=0 0 0
- joint joint_2_caster_10: origin xyz=0.038 -0.033293458 0.080377519 rpy=0 0 0 -> xyz=0.0357 -0.033293458 0.080377519 rpy=0 0 0
- joint joint_2_caster_11: origin xyz=0.038 -0.080377519 0.033293458 rpy=0 0 0 -> xyz=0.0357 -0.080377519 0.033293458 rpy=0 0 0
- joint joint_2_caster_12: origin xyz=0.038 -0.080377519 -0.033293458 rpy=0 0 0 -> xyz=0.0357 -0.080377519 -0.033293458 rpy=0 0 0
- joint joint_2_caster_13: origin xyz=0.038 -0.033293458 -0.080377519 rpy=0 0 0 -> xyz=0.0357 -0.033293458 -0.080377519 rpy=0 0 0
- joint joint_2_caster_14: origin xyz=0.038 0.033293458 -0.080377519 rpy=0 0 0 -> xyz=0.0357 0.033293458 -0.080377519 rpy=0 0 0
- joint joint_2_caster_15: origin xyz=0.038 0.080377519 -0.033293458 rpy=0 0 0 -> xyz=0.0357 0.080377519 -0.033293458 rpy=0 0 0
- joint joint_2_caster_2: origin xyz=0.038 0.0 0.087 rpy=0 0 0 -> xyz=0.0357 0.0 0.087 rpy=0 0 0
- joint joint_2_caster_3: origin xyz=0.038 -0.061518290 0.061518290 rpy=0 0 0 -> xyz=0.0357 -0.061518290 0.061518290 rpy=0 0 0
- joint joint_2_caster_4: origin xyz=0.038 -0.087 0.0 rpy=0 0 0 -> xyz=0.0357 -0.087 0.0 rpy=0 0 0
- joint joint_2_caster_5: origin xyz=0.038 -0.061518290 -0.061518290 rpy=0 0 0 -> xyz=0.0357 -0.061518290 -0.061518290 rpy=0 0 0
- joint joint_2_caster_6: origin xyz=0.038 0.0 -0.087 rpy=0 0 0 -> xyz=0.0357 0.0 -0.087 rpy=0 0 0
- joint joint_2_caster_7: origin xyz=0.038 0.061518290 -0.061518290 rpy=0 0 0 -> xyz=0.0357 0.061518290 -0.061518290 rpy=0 0 0
- joint joint_2_caster_8: origin xyz=0.038 0.080377519 0.033293458 rpy=0 0 0 -> xyz=0.0357 0.080377519 0.033293458 rpy=0 0 0
- joint joint_2_caster_9: origin xyz=0.038 0.033293458 0.080377519 rpy=0 0 0 -> xyz=0.0357 0.033293458 0.080377519 rpy=0 0 0
- joint joint_3_caster_0: origin xyz=-0.038 0.087 0.0 rpy=0 0 0 -> xyz=-0.0357 0.087 0.0 rpy=0 0 0
- joint joint_3_caster_1: origin xyz=-0.038 0.061518290 0.061518290 rpy=0 0 0 -> xyz=-0.0357 0.061518290 0.061518290 rpy=0 0 0
- joint joint_3_caster_10: origin xyz=-0.038 -0.033293458 0.080377519 rpy=0 0 0 -> xyz=-0.0357 -0.033293458 0.080377519 rpy=0 0 0
- joint joint_3_caster_11: origin xyz=-0.038 -0.080377519 0.033293458 rpy=0 0 0 -> xyz=-0.0357 -0.080377519 0.033293458 rpy=0 0 0
- joint joint_3_caster_12: origin xyz=-0.038 -0.080377519 -0.033293458 rpy=0 0 0 -> xyz=-0.0357 -0.080377519 -0.033293458 rpy=0 0 0
- joint joint_3_caster_13: origin xyz=-0.038 -0.033293458 -0.080377519 rpy=0 0 0 -> xyz=-0.0357 -0.033293458 -0.080377519 rpy=0 0 0
- joint joint_3_caster_14: origin xyz=-0.038 0.033293458 -0.080377519 rpy=0 0 0 -> xyz=-0.0357 0.033293458 -0.080377519 rpy=0 0 0
- joint joint_3_caster_15: origin xyz=-0.038 0.080377519 -0.033293458 rpy=0 0 0 -> xyz=-0.0357 0.080377519 -0.033293458 rpy=0 0 0
- joint joint_3_caster_2: origin xyz=-0.038 0.0 0.087 rpy=0 0 0 -> xyz=-0.0357 0.0 0.087 rpy=0 0 0
- joint joint_3_caster_3: origin xyz=-0.038 -0.061518290 0.061518290 rpy=0 0 0 -> xyz=-0.0357 -0.061518290 0.061518290 rpy=0 0 0
- joint joint_3_caster_4: origin xyz=-0.038 -0.087 0.0 rpy=0 0 0 -> xyz=-0.0357 -0.087 0.0 rpy=0 0 0
- joint joint_3_caster_5: origin xyz=-0.038 -0.061518290 -0.061518290 rpy=0 0 0 -> xyz=-0.0357 -0.061518290 -0.061518290 rpy=0 0 0
- joint joint_3_caster_6: origin xyz=-0.038 0.0 -0.087 rpy=0 0 0 -> xyz=-0.0357 0.0 -0.087 rpy=0 0 0
- joint joint_3_caster_7: origin xyz=-0.038 0.061518290 -0.061518290 rpy=0 0 0 -> xyz=-0.0357 0.061518290 -0.061518290 rpy=0 0 0
- joint joint_3_caster_8: origin xyz=-0.038 0.080377519 0.033293458 rpy=0 0 0 -> xyz=-0.0357 0.080377519 0.033293458 rpy=0 0 0
- joint joint_3_caster_9: origin xyz=-0.038 0.033293458 0.080377519 rpy=0 0 0 -> xyz=-0.0357 0.033293458 0.080377519 rpy=0 0 0

Commit message: temp

File: urdf/model.urdf (robot description, URDF)
Before this commit: robot trigger_a, 52 links, 51 joints
Joints:
- joint joint_2: axis 1 0 0 -> -1 0 0; origin xyz=0.14475 -0.25071 0.103 rpy=0 0 -1.0472 -> xyz=-0.2895 0 0.103 rpy=0 0 0
- joint joint_2_caster_0: origin xyz=0.0357 0.087 0.0 rpy=0 0 0 -> xyz=-0.0357 0.087 0.0 rpy=0 0 0
- joint joint_2_caster_1: origin xyz=0.0357 0.061518290 0.061518290 rpy=0 0 0 -> xyz=-0.0357 0.061518290 0.061518290 rpy=0 0 0
- joint joint_2_caster_10: origin xyz=0.0357 -0.033293458 0.080377519 rpy=0 0 0 -> xyz=-0.0357 -0.033293458 0.080377519 rpy=0 0 0
- joint joint_2_caster_11: origin xyz=0.0357 -0.080377519 0.033293458 rpy=0 0 0 -> xyz=-0.0357 -0.080377519 0.033293458 rpy=0 0 0
- joint joint_2_caster_12: origin xyz=0.0357 -0.080377519 -0.033293458 rpy=0 0 0 -> xyz=-0.0357 -0.080377519 -0.033293458 rpy=0 0 0
- joint joint_2_caster_13: origin xyz=0.0357 -0.033293458 -0.080377519 rpy=0 0 0 -> xyz=-0.0357 -0.033293458 -0.080377519 rpy=0 0 0
- joint joint_2_caster_14: origin xyz=0.0357 0.033293458 -0.080377519 rpy=0 0 0 -> xyz=-0.0357 0.033293458 -0.080377519 rpy=0 0 0
- joint joint_2_caster_15: origin xyz=0.0357 0.080377519 -0.033293458 rpy=0 0 0 -> xyz=-0.0357 0.080377519 -0.033293458 rpy=0 0 0
- joint joint_2_caster_2: origin xyz=0.0357 0.0 0.087 rpy=0 0 0 -> xyz=-0.0357 0.0 0.087 rpy=0 0 0
- joint joint_2_caster_3: origin xyz=0.0357 -0.061518290 0.061518290 rpy=0 0 0 -> xyz=-0.0357 -0.061518290 0.061518290 rpy=0 0 0
- joint joint_2_caster_4: origin xyz=0.0357 -0.087 0.0 rpy=0 0 0 -> xyz=-0.0357 -0.087 0.0 rpy=0 0 0
- joint joint_2_caster_5: origin xyz=0.0357 -0.061518290 -0.061518290 rpy=0 0 0 -> xyz=-0.0357 -0.061518290 -0.061518290 rpy=0 0 0
- joint joint_2_caster_6: origin xyz=0.0357 0.0 -0.087 rpy=0 0 0 -> xyz=-0.0357 0.0 -0.087 rpy=0 0 0
- joint joint_2_caster_7: origin xyz=0.0357 0.061518290 -0.061518290 rpy=0 0 0 -> xyz=-0.0357 0.061518290 -0.061518290 rpy=0 0 0
- joint joint_2_caster_8: origin xyz=0.0357 0.080377519 0.033293458 rpy=0 0 0 -> xyz=-0.0357 0.080377519 0.033293458 rpy=0 0 0
- joint joint_2_caster_9: origin xyz=0.0357 0.033293458 0.080377519 rpy=0 0 0 -> xyz=-0.0357 0.033293458 0.080377519 rpy=0 0 0
- joint joint_3: axis -1 0 0 -> 1 0 0; origin xyz=-0.2895 0 0.103 rpy=0 0 0 -> xyz=0.14475 -0.25071 0.103 rpy=0 0 -1.0472
- joint joint_3_caster_0: origin xyz=-0.0357 0.087 0.0 rpy=0 0 0 -> xyz=0.0357 0.087 0.0 rpy=0 0 0
- joint joint_3_caster_1: origin xyz=-0.0357 0.061518290 0.061518290 rpy=0 0 0 -> xyz=0.0357 0.061518290 0.061518290 rpy=0 0 0
- joint joint_3_caster_10: origin xyz=-0.0357 -0.033293458 0.080377519 rpy=0 0 0 -> xyz=0.0357 -0.033293458 0.080377519 rpy=0 0 0
- joint joint_3_caster_11: origin xyz=-0.0357 -0.080377519 0.033293458 rpy=0 0 0 -> xyz=0.0357 -0.080377519 0.033293458 rpy=0 0 0
- joint joint_3_caster_12: origin xyz=-0.0357 -0.080377519 -0.033293458 rpy=0 0 0 -> xyz=0.0357 -0.080377519 -0.033293458 rpy=0 0 0
- joint joint_3_caster_13: origin xyz=-0.0357 -0.033293458 -0.080377519 rpy=0 0 0 -> xyz=0.0357 -0.033293458 -0.080377519 rpy=0 0 0
- joint joint_3_caster_14: origin xyz=-0.0357 0.033293458 -0.080377519 rpy=0 0 0 -> xyz=0.0357 0.033293458 -0.080377519 rpy=0 0 0
- joint joint_3_caster_15: origin xyz=-0.0357 0.080377519 -0.033293458 rpy=0 0 0 -> xyz=0.0357 0.080377519 -0.033293458 rpy=0 0 0
- joint joint_3_caster_2: origin xyz=-0.0357 0.0 0.087 rpy=0 0 0 -> xyz=0.0357 0.0 0.087 rpy=0 0 0
- joint joint_3_caster_3: origin xyz=-0.0357 -0.061518290 0.061518290 rpy=0 0 0 -> xyz=0.0357 -0.061518290 0.061518290 rpy=0 0 0
- joint joint_3_caster_4: origin xyz=-0.0357 -0.087 0.0 rpy=0 0 0 -> xyz=0.0357 -0.087 0.0 rpy=0 0 0
- joint joint_3_caster_5: origin xyz=-0.0357 -0.061518290 -0.061518290 rpy=0 0 0 -> xyz=0.0357 -0.061518290 -0.061518290 rpy=0 0 0
- joint joint_3_caster_6: origin xyz=-0.0357 0.0 -0.087 rpy=0 0 0 -> xyz=0.0357 0.0 -0.087 rpy=0 0 0
- joint joint_3_caster_7: origin xyz=-0.0357 0.061518290 -0.061518290 rpy=0 0 0 -> xyz=0.0357 0.061518290 -0.061518290 rpy=0 0 0
- joint joint_3_caster_8: origin xyz=-0.0357 0.080377519 0.033293458 rpy=0 0 0 -> xyz=0.0357 0.080377519 0.033293458 rpy=0 0 0
- joint joint_3_caster_9: origin xyz=-0.0357 0.033293458 0.080377519 rpy=0 0 0 -> xyz=0.0357 0.033293458 0.080377519 rpy=0 0 0
